File: fred_v3/SENSORES.kicad_sch (KiCad schematic)
At the start: 12 parts, among them J7 Conn_01x04, J8 Conn_01x04, J9 Conn_01x04

Commit message: Add files via upload
Parts:
- added C67: 100nF, Capacitor_SMD:C_0603_1608Metric_Pad1.08x0.95mm_HandSolder, symbol Device:C
- added J30: Conn_01x04, Connector_JST:JST_EH_S4B-EH_1x04_P2.50mm_Horizontal, symbol Connector_Generic:Conn_01x04
- added J31: Conn_01x03, Connector_JST:JST_EH_S3B-EH_1x03_P2.50mm_Horizontal, symbol Connector_Generic:Conn_01x03
- added R117: Pull_Up Hall (Pode não ser necessário), Resistor_SMD:R_0603_1608Metric_Pad0.98x0.95mm_HandSolder, symbol Device:R
- C27, C28, C29: footprint (none) -> Capacitor_SMD:C_0603_1608Metric_Pad1.08x0.95mm_HandSolder
- J7, J8, J9: footprint (none) -> Connector_JST:JST_EH_S4B-EH_1x04_P2.50mm_Horizontal
- R30, R31, R32, R33, R34, R35: footprint (none) -> Resistor_SMD:R_0603_1608Metric_Pad0.98x0.95mm_HandSolder
Connections:
- net GND: now also C67.2, J30.2 (Pin_2), J31.2 (Pin_2)
- net 3,3V renamed 5V
- net 5V: now also C67.1, J30.1 (Pin_1), J31.1 (Pin_1), R117.1
- new net HALL_OUT: J31.3 (Pin_3), R117.2
- new net SCL: J30.3 (Pin_3)
- new net SDA: J30.4 (Pin_4)
Other:
- note added: "Add: Sensor de efeito Hall, sensor de cores, sensor de buraco (VL) e GPS para ir no serial do RASP"
- note added: "Sensor de Cores RGB"
- note added: "Sensor de Efeito Hall"
- note added: "Sensores Ultrassonicos"
- moved on the sheet: C27, C28, C29, J7, J8, J9, R30, R31, R32, R33, R34, R35
