File: fred_v3/Esp_1.kicad_sch (KiCad schematic)
At the start: 40 parts, among them J1 Conn_01x14, J2 Conn_01x13, J5 USB_C_Receptacle_USB2.0, Q1 SS8050-G, Q2 SS8050-G, Q3 Q_PMOS_GSD, SW1 SW_Push, SW2 SW_Push, U1 AMS1117-3.3, U2 CP2102N-Axx-xQFN28, U3 ESP32-WROOM-E

Commit message: Add files via upload
Parts:
- C1, C2: footprint (none) -> Capacitor_SMD:C_0603_1608Metric_Pad1.08x0.95mm_HandSolder
- C3: value 4.7uF/6.3V(10%) -> 4.7uF
- C4, C5, C6, C8, C9: value 0.1uF/50V(10%) -> 0.1uF
- C7: value 22uF/10V(20%) -> 22uF
- D1: footprint (none) -> LED_SMD:LED_1206_3216Metric_Pad1.42x1.75mm_HandSolder
- J5: footprint (none) -> Connector_USB:USB_C_Receptacle_GCT_USB4105-xx-A_16P_TopMnt_Horizontal
- R1, R21, R22, R23: footprint (none) -> Resistor_SMD:R_0603_1608Metric_Pad0.98x0.95mm_HandSolder
- R10: value 1k(5%) -> 1k
- R2, R3, R7: value 10k(5%) -> 10k
- R4: value 22.1k(5%) -> 22.1k
- R5: value 47.5k(5%) -> 47.5k
- R6: value 2k(5%) -> 2k
- R8: value 10K(10%) -> 10k
Connections:
- net 5V is gone; now on net 5V_USB: D3.1 (K)
- net 5V_USB: now also R4.1
- net VBUS: no longer R4.1
Changed lines of the file:
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@@
   (junction (at 162.56 148.59) (diameter 0) (color 0 0 0 0)
+  )
+  (junction (at 250.19 152.4) (diameter 0) (color 0 0 0 0)
   )
   (junction (at 231.14 149.86) (diameter 0) (color 0 0 0 0)
@@
     (stroke (width 0) (type default))
   )
+  (wire (pts (xy 247.65 156.21) (xy 250.19 156.21))
+    (stroke (width 0) (type default))
+  )
   (wire (pts (xy 328.93 154.94) (xy 327.66 154.94))
     (stroke (width 0) (type default))
@@
     (stroke (width 0) (type default))
   )
+  (wire (pts (xy 250.19 152.4) (xy 251.46 152.4))
+    (stroke (width 0) (type default))
+  )
   (wire (pts (xy 76.2 66.04) (xy 76.2 64.77))
     (stroke (width 0) (type default))
@@
     (stroke (width 0) (type default))
   )
+  (wire (pts (xy 250.19 156.21) (xy 250.19 152.4))
+    (stroke (width 0) (type default))
+  )
   (wire (pts (xy 68.58 184.15) (xy 68.58 209.55))
     (stroke (width 0) (type default))
@@
     (stroke (width 0) (type default))
   )
-  (wire (pts (xy 248.92 152.4) (xy 251.46 152.4))
+  (wire (pts (xy 248.92 152.4) (xy 250.19 152.4))
     (stroke (width 0) (type default))
   )
@@
     )
   )
-  (global_label "VBUS" (shape input) (at 128.27 195.58 90) (fields_autoplaced)
-    (effects (font (size 1.27 1.27)) (justify left))
-    (property "Intersheetrefs" "${INTERSHEET_REFS}" (at 128.27 187.6962 90)
-      (effects (font (size 1.27 1.27)) (justify left) hide)
-    )
-  )
   (global_label "VBUS_CP210" (shape input) (at 132.08 213.36 0) (fields_autoplaced)
     (effects (font (size 1.27 1.27)) (justify left))
@@
     )
   )
+  (global_label "5V_USB" (shape input) (at 128.27 195.58 90) (fields_autoplaced)
+    (effects (font (size 1.27 1.27)) (justify left))
+    (property "Intersheetrefs" "${INTERSHEET_REFS}" (at 128.27 185.5191 90)
+      (effects (font (size 1.27 1.27)) (justify left) hide)
+    )
+  )
   (global_label "IO35" (shape input) (at 381 194.31 0) (fields_autoplaced)
     (effects (font (size 1.27 1.27)) (justify left))
@@
     )
   )
+  (global_label "5V_USB" (shape input) (at 100.33 156.21 0) (fields_autoplaced)
+    (effects (font (size 1.27 1.27)) (justify left))
+    (property "Intersheetrefs" "${INTERSHEET_REFS}" (at 110.3909 156.21 0)
+      (effects (font (size 1.27 1.27)) (justify left) hide)
+    )
+  )
   (global_label "DTR" (shape input) (at 179.07 171.45 0) (fields_autoplaced)
     (effects (font (size 1.27 1.27)) (justify left))
@@
     )
   )
-  (global_label "5V" (shape input) (at 100.33 156.21 0) (fields_autoplaced)
-    (effects (font (size 1.27 1.27)) (justify left))
-    (property "Intersheetrefs" "${INTERSHEET_REFS}" (at 105.6133 156.21 0)
-      (effects (font (size 1.27 1.27)) (justify left) hide)
-    )
-  )
   (global_label "RTS" (shape input) (at 179.07 163.83 0) (fields_autoplaced)
     (effects (font (size 1.27 1.27)) (justify left))
@@
   (hierarchical_label "SCL" (shape input) (at 344.17 148.59 90) (fields_autoplaced)
     (effects (font (size 1.27 1.27)) (justify left))
+  )
+  (hierarchical_label "HALL_IN" (shape input) (at 247.65 156.21 180) (fields_autoplaced)
+    (effects (font (size 1.27 1.27)) (justify right))
   )
   (hierarchical_label "MPU_INT" (shape input) (at 330.2 144.78 0) (fields_autoplaced)
@@
       (effects (font (size 1.27 1.27)) (justify left))
     )
-    (property "Value" "0.1uF/50V(10%)" (at 290.83 104.14 90)
+    (property "Value" "0.1uF" (at 290.83 104.14 90)
       (effects (font (size 1.27 1.27)) (justify left))
     )
@@
       (effects (font (size 1.27 1.27)) (justify left))
     )
-    (property "Footprint" "" (at 23.622 201.93 90)
+    (property "Footprint" "Resistor_SMD:R_0603_1608Metric_Pad0.98x0.95mm_HandSolder" (at 23.622 201.93 90)
       (effects (font (size 1.27 1.27)) hide)
     )
@@
       (effects (font (size 1.27 1.27)) (justify left))
     )
-    (property "Value" "1k(5%)" (at 73.66 63.5 90)
+    (property "Value" "1k" (at 73.66 63.5 90)
       (effects (font (size 1.27 1.27)) (justify left))
     )
@@
       (effects (font (size 1.27 1.27)) (justify left))
     )
-    (property "Value" "0.1uF/50V(10%)" (at 124.46 171.45 90)
+    (property "Value" "0.1uF" (at 124.46 171.45 90)
       (effects (font (size 1.27 1.27)) (justify left))
     )
@@
       (effects (font (size 1.27 1.27)) (justify left))
     )
-    (property "Value" "10K(10%)" (at 234.95 114.3 0)
+    (property "Value" "10k" (at 234.95 114.3 0)
       (effects (font (size 1.27 1.27)) (justify left))
     )
@@
       (effects (font (size 1.27 1.27)) (justify left))
     )
-    (property "Value" "2k(5%)" (at 143.51 157.48 90)
+    (property "Value" "2k" (at 146.05 156.21 90)
       (effects (font (size 1.27 1.27)) (justify left))
     )
@@
       (effects (font (size 1.27 1.27)) (justify left))
     )
-    (property "Value" "0.1uF/50V(10%)" (at 365.76 135.89 90)
+    (property "Value" "0.1uF" (at 365.76 135.89 90)
       (effects (font (size 1.27 1.27)) (justify left))
     )
@@
       (effects (font (size 1.27 1.27)) (justify left))
     )
-    (property "Value" "0.1uF/50V(10%)" (at 365.76 110.49 90)
+    (property "Value" "0.1uF" (at 365.76 110.49 90)
       (effects (font (size 1.27 1.27)) (justify left))
     )
@@
       (effects (font (size 1.27 1.27)) (justify left))
     )
-    (property "Footprint" "" (at 52.832 193.04 90)
+    (property "Footprint" "Resistor_SMD:R_0603_1608Metric_Pad0.98x0.95mm_HandSolder" (at 52.832 193.04 90)
       (effects (font (size 1.27 1.27)) hide)
     )
@@
       (effects (font (size 1.27 1.27)) (justify left))
     )
-    (property "Footprint" "" (at 89.662 59.69 90)
+    (property "Footprint" "Resistor_SMD:R_0603_1608Metric_Pad0.98x0.95mm_HandSolder" (at 89.662 59.69 90)
       (effects (font (size 1.27 1.27)) hide)
     )
@@
       (effects (font (size 1.27 1.27)) (justify left))
     )
-    (property "Value" "47.5k(5%)" (at 125.73 222.25 90)
+    (property "Value" "47.5k" (at 125.73 222.25 90)
       (effects (font (size 1.27 1.27)) (justify left))
     )
@@
       (effects (font (size 1.27 1.27)))
     )
-    (property "Value" "10k(5%)" (at 81.28 236.22 90)
+    (property "Value" "10k" (at 81.28 236.22 90)
       (effects (font (size 1.27 1.27)))
     )
@@
       (effects (font (size 1.27 1.27)))
     )
-    (property "Value" "10k(5%)" (at 81.28 256.54 90)
+    (property "Value" "10k" (at 81.28 256.54 90)
       (effects (font (size 1.27 1.27)))
     )
@@
       (effects (font (size 1.27 1.27)) (justify left))
     )
-    (property "Value" "22uF/10V(20%)" (at 303.53 102.87 90)
+    (property "Value" "22uF" (at 303.53 102.87 90)
       (effects (font (size 1.27 1.27)) (justify left))
     )
@@
       (effects (font (size 1.27 1.27)) (justify left))
     )
-    (property "Footprint" "" (at 59.182 193.04 90)
+    (property "Footprint" "Resistor_SMD:R_0603_1608Metric_Pad0.98x0.95mm_HandSolder" (at 59.182 193.04 90)
       (effects (font (size 1.27 1.27)) hide)
     )
@@
       (effects (font (size 1.27 1.27)) (justify left))
     )
-    (property "Footprint" "" (at 102.5652 68.58 0)
+    (property "Footprint" "Capacitor_SMD:C_0603_1608Metric_Pad1.08x0.95mm_HandSolder" (at 102.5652 68.58 0)
       (effects (font (size 1.27 1.27)) hide)
     )
@@
       (effects (font (size 1.27 1.27)) (justify left))
     )
-    (property "Value" "10k(5%)" (at 184.15 195.58 90)
+    (property "Value" "10k" (at 184.15 195.58 90)
       (effects (font (size 1.27 1.27)) (justify left))
     )
@@
       (effects (font (size 1.27 1.27)) (justify left))
     )
-    (property "Footprint" "" (at 136.8552 68.58 0)
+    (property "Footprint" "Capacitor_SMD:C_0603_1608Metric_Pad1.08x0.95mm_HandSolder" (at 136.8552 68.58 0)
       (effects (font (size 1.27 1.27)) hide)
     )
@@
       (effects (font (size 1.27 1.27)))
     )
-    (property "Footprint" "" (at 36.83 171.45 0)
+    (property "Footprint" "Connector_USB:USB_C_Receptacle_GCT_USB4105-xx-A_16P_TopMnt_Horizontal" (at 36.83 171.45 0)
       (effects (font (size 1.27 1.27)) hide)
     )
@@
       (effects (font (size 1.27 1.27)) (justify left))
     )
-    (property "Value" "0.1uF/50V(10%)" (at 228.6 135.89 90)
+    (property "Value" "0.1uF" (at 228.6 135.89 90)
       (effects (font (size 1.27 1.27)) (justify left))
     )
@@
       (effects (font (size 1.27 1.27)) (justify left))
     )
-    (property "Value" "22.1k(5%)" (at 125.73 209.55 90)
+    (property "Value" "22.1k" (at 125.73 209.55 90)
       (effects (font (size 1.27 1.27)) (justify left))
     )
@@
       (effects (font (size 1.27 1.27)) (justify right))
     )
-    (property "Footprint" "" (at 91.44 69.85 0)
+    (property "Footprint" "LED_SMD:LED_1206_3216Metric_Pad1.42x1.75mm_HandSolder" (at 91.44 69.85 0)
       (effects (font (size 1.27 1.27)) hide)
     )
@@
       (effects (font (size 1.27 1.27)) (justify left))
     )
-    (property "Value" "4.7uF/6.3V(10%)" (at 113.03 171.45 90)
-      (effects (font (size 1.27 1.27)) (justify left))
-    )
+    (property "Value" "4.7uF" (at 113.03 171.45 90)
+      (effects (font (size 1.27 1.27)) (justify left))
+    )

Commit message: Add files via upload
Parts:
- removed J1: Conn_01x14, Connector_PinHeader_2.54mm:PinHeader_1x14_P2.54mm_Vertical, symbol Connector_Generic:Conn_01x14
- removed J2: Conn_01x13, Connector_PinHeader_2.54mm:PinHeader_1x13_P2.54mm_Vertical, symbol Connector_Generic:Conn_01x13
- removed R21: R, Resistor_SMD:R_0603_1608Metric_Pad0.98x0.95mm_HandSolder, symbol Device:R
Connections:
- net RXD0 is gone; now on net RXD_ESP1: U3.35 (U0TXD/GPIO1)
- net TXD0 is gone; now on net TXD_EPS1: U3.34 (U0RXD/GPIO3)
- net 5V_USB renamed 5V_USB_ESP1
- net D+ renamed D+_ESP1
- net D- renamed D-_ESP1
- net DTR renamed DTR_ESP1
- net EN renamed EN_ESP1
- net EXT_5V renamed EXT_5V_1
- net IO0 renamed IO0_ESP1
- net IO12 renamed IO12_ESP1
- net IO13 renamed IO13_ESP1
- net IO14 renamed IO14_ESP1
- net IO15 renamed IO15_ESP1
- net IO16 renamed IO16_ESP1
- net IO17 renamed IO17_ESP1
- net IO18 renamed IO18_ESP1
- net IO19 renamed IO19_ESP1
- net IO2 renamed IO2_ESP1
- net IO21 renamed IO21_ESP1
- net IO22 renamed IO22_ESP1
- net IO23 renamed IO23_ESP1
- net IO25 renamed IO25_ESP1
- net IO26 renamed IO26_ESP1
- net IO27 renamed IO27_ESP1
- net IO32 renamed IO32_ESP1
- net IO33 renamed IO33_ESP1
- net IO34 renamed IO34_ESP1
- net IO35 renamed IO35_ESP1
- net IO36 renamed IO36_ESP1
- net IO39 renamed IO39_ESP1
- net IO4 renamed IO4_ESP1
- net IO5 renamed IO5_ESP1
- net RTS renamed RTS_ESP1
- net RXD renamed RXD_ESP1
- net TXD renamed TXD_EPS1
- net VBUS renamed VBUS_ESP1
- net VBUS_CP210 renamed VBUS_CP210_ESP1
- no-connect marks 17 -> 18
Other:
- moved on the sheet: C5
