File: fred_v3/LED_LVL_SHIFTER.kicad_sch (KiCad schematic)
At the start: 3 parts, among them U10 AD8001AN

Commit message: Add files via upload
Parts:
- R36, R37: footprint (none) -> Resistor_SMD:R_0603_1608Metric_Pad0.98x0.95mm_HandSolder
Changed lines of the file:
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@@
 (kicad_sch (version 20230121) (generator eeschema)
   (paper "A4")
+  (title_block
+    (rev "1")
+  )
   (junction (at 133.35 104.14) (diameter 0) (color 0 0 0 0)
   )
@@
       (effects (font (size 1.27 1.27)))
     )
-    (property "Footprint" "" (at 128.27 105.918 90)
+    (property "Footprint" "Resistor_SMD:R_0603_1608Metric_Pad0.98x0.95mm_HandSolder" (at 128.27 105.918 90)
       (effects (font (size 1.27 1.27)) hide)
     )
@@
       (effects (font (size 1.27 1.27)) (justify left))
     )
-    (property "Footprint" "" (at 131.572 109.22 90)
+    (property "Footprint" "Resistor_SMD:R_0603_1608Metric_Pad0.98x0.95mm_HandSolder" (at 131.572 109.22 90)
       (effects (font (size 1.27 1.27)) hide)
     )

Commit message: Add files via upload
Parts:
- U10: value AD8001AN -> 741
Changed lines of the file:
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@@
   (symbol (lib_id "Amplifier_Operational:AD8001AN") (at 144.78 99.06 0) (unit 1)
     (in_bom yes) (on_board yes) (dnp no) (fields_autoplaced)
-    (property "Reference" "U10" (at 156.21 94.8691 0)
+    (property "Reference" "U10" (at 153.67 94.8691 0)
       (effects (font (size 1.27 1.27)))
     )
-    (property "Value" "AD8001AN" (at 156.21 97.4091 0)
+    (property "Value" "741" (at 153.67 97.4091 0)
       (effects (font (size 1.27 1.27)))
     )
