File: fred_v3/Esp_2.kicad_sch (KiCad schematic)
At the start: 40 parts, among them J3 Conn_01x14, J4 Conn_01x13, J5 USB_C_Receptacle_USB2.0, Q1 SS8050-G, Q2 SS8050-G, Q3 Q_PMOS_GSD, SW1 SW_Push, SW2 SW_Push, U1 AMS1117-3.3, U2 CP2102N-Axx-xQFN28, U3 ESP32-WROOM-E

Commit message: Add files via upload
Changed lines of the file:
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@@
     (stroke (width 0) (type default))
   )
-  (wire (pts (xy 232.41 167.64) (xy 232.41 168.91))
+  (wire (pts (xy 280.67 170.18) (xy 280.67 171.45))
     (stroke (width 0) (type default))
   )
@@
     )
   )
-  (hierarchical_label "GND" (shape output) (at 232.41 167.64 90) (fields_autoplaced)
+  (hierarchical_label "GND" (shape output) (at 280.67 170.18 90) (fields_autoplaced)
     (effects (font (size 1.27 1.27)) (justify left))
   )
@@
     )
   )
-  (symbol (lib_id "power:GND") (at 232.41 168.91 0) (unit 1)
+  (symbol (lib_id "power:GND") (at 280.67 171.45 0) (unit 1)
     (in_bom yes) (on_board yes) (dnp no)
-    (property "Reference" "#PWR015" (at 232.41 175.26 0)
-      (effects (font (size 1.27 1.27)) hide)
-    )
-    (property "Value" "GND" (at 233.68 156.21 0)
-      (effects (font (size 1.27 1.27)))
-    )
-    (property "Footprint" "" (at 232.41 168.91 0)
-      (effects (font (size 1.27 1.27)) hide)
-    )
-    (property "Datasheet" "" (at 232.41 168.91 0)
-      (effects (font (size 1.27 1.27)) hide)
-    )
+    (property "Reference" "#PWR015" (at 280.67 177.8 0)
+      (effects (font (size 1.27 1.27)) hide)
+    )
+    (property "Value" "GND" (at 280.67 176.53 0)
+      (effects (font (size 1.27 1.27)))
+    )
+    (property "Footprint" "" (at 280.67 171.45 0)
+      (effects (font (size 1.27 1.27)) hide)
+    )
+    (property "Datasheet" "" (at 280.67 171.45 0)
+      (effects (font (size 1.27 1.27)) hide)
+    )

Commit message: Add files via upload
Parts:
- C1, C2: footprint (none) -> Capacitor_SMD:C_0603_1608Metric_Pad1.08x0.95mm_HandSolder
- C3: value 4.7uF/6.3V(10%) -> 4.7uF
- C4, C5, C6, C8, C9: value 0.1uF/50V(10%) -> 0.1uF
- C7: value 22uF/10V(20%) -> 22uF
- D1: footprint (none) -> LED_SMD:LED_1206_3216Metric_Pad1.42x1.75mm_HandSolder
- J5: footprint (none) -> Connector_USB:USB_C_Receptacle_GCT_USB4105-xx-A_16P_TopMnt_Horizontal
- R1, R21, R22, R23: footprint (none) -> Resistor_SMD:R_0603_1608Metric_Pad0.98x0.95mm_HandSolder
- R10: value 1k(5%) -> 1k
- R2, R3, R7: value 10k(5%) -> 10k
- R4: value 22.1k(5%) -> 22.1k
- R5: value 47.5k(5%) -> 47.5k
- R6: value 2k(5%) -> 2k
- R8: value 10K(10%) -> 10k
Connections:
- net 5V is gone; now on net 5V_USB: D3.1 (K)
- net 5V_USB: now also R4.1
- net VBUS: no longer R4.1
Other:
- moved on the sheet: C5, C8, C9, R8, SW1, SW2

Commit message: Add files via upload
Parts:
- removed J3: Conn_01x14, Connector_PinHeader_2.54mm:PinHeader_1x14_P2.54mm_Vertical, symbol Connector_Generic:Conn_01x14
- removed J4: Conn_01x13, Connector_PinHeader_2.54mm:PinHeader_1x13_P2.54mm_Vertical, symbol Connector_Generic:Conn_01x13
- removed R21: R, Resistor_SMD:R_0603_1608Metric_Pad0.98x0.95mm_HandSolder, symbol Device:R
Connections:
- net TXD is gone; now on net TXD_ESP2: U2.26 (TXD)
- net TXD0 is gone; now on net RXD_ESP2: U3.34 (U0RXD/GPIO3)
- net 3.3V renamed 3,3V_ESP2
- net 5V_USB renamed 5V_USB_ESP2
- net D+ renamed D+_ESP2
- net D- renamed D-_ESP2
- net DTR renamed DTR_ESP2
- net EN renamed EN_ESP2
- net EXT_5V renamed EXT_5V_2
- net IO0 renamed IO0_ESP2
- net IO12 renamed IO12_ESP2
- net IO13 renamed IO13_ESP2
- net IO14 renamed IO14_ESP2
- net IO15 renamed IO15_ESP2
- net IO16 renamed IO16_ESP2
- net IO17 renamed IO17_ESP2
- net IO18 renamed IO18_ESP2
- net IO19 renamed IO19_ESP2
- net IO2 renamed IO2_ESP2
- net IO21 renamed IO21_ESP2
- net IO22 renamed IO22_ESP2
- net IO23 renamed IO23_ESP2
- net IO25 renamed IO25_ESP2
- net IO26 renamed IO26_ESP2
- net IO27 renamed IO27_ESP2
- net IO32 renamed IO32_ESP2
- net IO33 renamed IO33_ESP2
- net IO34 renamed IO34_ESP2
- net IO35 renamed IO35_ESP2
- net IO36 renamed IO36_ESP2
- net IO39 renamed IO39_ESP2
- net IO4 renamed IO4_ESP2
- net IO5 renamed IO5_ESP2
- net RTS renamed RTS_ESP2
- net RXD renamed RXD_ESP2
- net RXD0 renamed TXD_ESP2
- net VBUS renamed VBUS_ESP2
- net VBUS_CP210 renamed VBUS_CP210_ESP2
- no-connect marks 17 -> 18

Commit message: Add files via upload
Connections:
- net EN_ESP2: no longer C8.2, Q1.2 (C), SW1.2
- net 3,3V_ESP2 renamed 3,3V_ESP3
- net 5V_USB_ESP2 renamed 5V_USB_ESP3
- net D+_ESP2 renamed D+_ESP3
- net D-_ESP2 renamed D-_ESP3
- net DTR_ESP2 renamed DTR_ESP3
- net EXT_5V_2 renamed EXT_5V_3
- net IO0_ESP2 renamed IO0_ESP3
- net IO12_ESP2 renamed IO12_ESP3
- net IO13_ESP2 renamed IO13_ESP3
- net IO14_ESP2 renamed IO14_ESP3
- net IO15_ESP2 renamed IO15_ESP3
- net IO16_ESP2 renamed IO16_ESP3
- net IO17_ESP2 renamed IO17_ESP3
- net IO18_ESP2 renamed IO18_ESP3
- net IO19_ESP2 renamed IO19_ESP3
- net IO21_ESP2 renamed IO21_ESP3
- net IO22_ESP2 renamed IO22_ESP3
- net IO23_ESP2 renamed IO23_ESP3
- net IO25_ESP2 renamed IO25_ESP3
- net IO26_ESP2 renamed IO26_ESP3
- net IO27_ESP2 renamed IO27_ESP3
- net IO2_ESP2 renamed IO2_ESP3
- net IO32_ESP2 renamed IO32_ESP3
- net IO33_ESP2 renamed IO33_ESP3
- net IO34_ESP2 renamed IO34_ESP3
- net IO35_ESP2 renamed IO35_ESP3
- net IO36_ESP2 renamed IO36_ESP3
- net IO39_ESP2 renamed IO39_ESP3
- net IO4_ESP2 renamed IO4_ESP3
- net IO5_ESP2 renamed IO5_ESP3
- net RTS_ESP2 renamed RTS_ESP3
- net RXD_ESP2 renamed RXD_ESP3
- net TXD_ESP2 renamed TXD_ESP3
- net VBUS_CP210_ESP2 renamed VBUS_CP210_ESP3
- net VBUS_ESP2 renamed VBUS_ESP3
- new net EN_ESP3: C8.2, Q1.2 (C), SW1.2
