File: fred_v3/Lógica.kicad_sch (KiCad schematic)
At the start: 3 parts, among them J10 Conn_01x03

Commit message: Add files via upload
Connections:
- net LED_LVL_SHIFTER/GND renamed GND
Changed lines of the file:
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@@
   (junction (at 72.39 85.09) (diameter 0) (color 0 0 0 0)
   )
+  (junction (at 205.74 105.41) (diameter 0) (color 0 0 0 0)
+  )
   (junction (at 74.93 86.36) (diameter 0) (color 0 0 0 0)
   )
@@
   (junction (at 144.78 104.14) (diameter 0) (color 0 0 0 0)
   )
+  (junction (at 74.93 78.74) (diameter 0) (color 0 0 0 0)
+  )
+  (junction (at 81.28 158.75) (diameter 0) (color 0 0 0 0)
+  )
   (wire (pts (xy 96.52 101.6) (xy 99.06 101.6))
     (stroke (width 0) (type default))
@@
     (stroke (width 0) (type default))
   )
+  (wire (pts (xy 205.74 105.41) (xy 208.28 105.41))
+    (stroke (width 0) (type default))
+  )
   (wire (pts (xy 138.43 106.68) (xy 138.43 133.35))
     (stroke (width 0) (type default))
@@
     (stroke (width 0) (type default))
   )
+  (wire (pts (xy 81.28 158.75) (xy 81.28 161.29))
+    (stroke (width 0) (type default))
+  )
+  (wire (pts (xy 49.53 95.25) (xy 49.53 82.55))
+    (stroke (width 0) (type default))
+  )
+  (wire (pts (xy 205.74 86.36) (xy 205.74 102.87))
+    (stroke (width 0) (type default))
+  )
+  (wire (pts (xy 203.2 105.41) (xy 205.74 105.41))
+    (stroke (width 0) (type default))
+  )
   (wire (pts (xy 74.93 86.36) (xy 96.52 86.36))
     (stroke (width 0) (type default))
@@
     (stroke (width 0) (type default))
   )
+  (wire (pts (xy 205.74 102.87) (xy 208.28 102.87))
+    (stroke (width 0) (type default))
+  )
   (wire (pts (xy 92.71 157.48) (xy 92.71 148.59))
     (stroke (width 0) (type default))
   )
-  (wire (pts (xy 57.15 158.75) (xy 93.98 158.75))
+  (wire (pts (xy 57.15 158.75) (xy 81.28 158.75))
     (stroke (width 0) (type default))
   )
@@
     (stroke (width 0) (type default))
   )
+  (wire (pts (xy 81.28 158.75) (xy 93.98 158.75))
+    (stroke (width 0) (type default))
+  )
   (wire (pts (xy 57.15 143.51) (xy 59.69 143.51))
     (stroke (width 0) (type default))
@@
     (stroke (width 0) (type default))
   )
+  (wire (pts (xy 74.93 78.74) (xy 74.93 86.36))
+    (stroke (width 0) (type default))
+  )
+  (wire (pts (xy 52.07 95.25) (xy 49.53 95.25))
+    (stroke (width 0) (type default))
+  )
+  (wire (pts (xy 74.93 78.74) (xy 83.82 78.74))
+    (stroke (width 0) (type default))
+  )
+  (wire (pts (xy 29.845 173.355) (xy 29.845 177.165))
+    (stroke (width 0) (type default))
+  )
   (wire (pts (xy 119.38 106.68) (xy 138.43 106.68))
     (stroke (width 0) (type default))
   )
+  (wire (pts (xy 205.74 105.41) (xy 205.74 137.16))
+    (stroke (width 0) (type default))
+  )
   (wire (pts (xy 57.15 148.59) (xy 57.15 158.75))
     (stroke (width 0) (type default))
@@
     (stroke (width 0) (type default))
   )
-  (wire (pts (xy 74.93 69.85) (xy 74.93 86.36))
+  (wire (pts (xy 74.93 69.85) (xy 74.93 78.74))
     (stroke (width 0) (type default))
   )
@@
   (wire (pts (xy 43.18 109.22) (xy 52.07 109.22))
     (stroke (width 0) (type default))
+  )
+  (global_label "GND" (shape input) (at 81.28 161.29 270) (fields_autoplaced)
+    (effects (font (size 1.27 1.27)) (justify right))
+    (property "Intersheetrefs" "${INTERSHEET_REFS}" (at 81.28 168.1457 90)
+      (effects (font (size 1.27 1.27)) (justify right) hide)
+    )
+  )
+  (global_label "GND" (shape input) (at 29.845 177.165 270) (fields_autoplaced)
+    (effects (font (size 1.27 1.27)) (justify right))
+    (property "Intersheetrefs" "${INTERSHEET_REFS}" (at 29.845 184.0207 90)
+      (effects (font (size 1.27 1.27)) (justify right) hide)
+    )
+  )
+  (global_label "GND" (shape input) (at 83.82 78.74 0) (fields_autoplaced)
+    (effects (font (size 1.27 1.27)) (justify left))
+    (property "Intersheetrefs" "${INTERSHEET_REFS}" (at 90.6757 78.74 0)
+      (effects (font (size 1.27 1.27)) (justify left) hide)
+    )
+  )
+  (global_label "GND" (shape input) (at 205.74 137.16 270) (fields_autoplaced)
+    (effects (font (size 1.27 1.27)) (justify right))
+    (property "Intersheetrefs" "${INTERSHEET_REFS}" (at 205.74 144.0157 90)
+      (effects (font (size 1.27 1.27)) (justify right) hide)
+    )
+  )
+  (hierarchical_label "Esp1_5V" (shape input) (at 49.53 82.55 90) (fields_autoplaced)
+    (effects (font (size 1.27 1.27)) (justify left))
+  )
+  (hierarchical_label "Esp2_5V" (shape input) (at 205.74 86.36 90) (fields_autoplaced)
+    (effects (font (size 1.27 1.27)) (justify left))
+  )
+  (hierarchical_label "GND" (shape input) (at 29.845 173.355 90) (fields_autoplaced)
+    (effects (font (size 1.27 1.27)) (justify left))
   )
   (hierarchical_label "CANH" (shape input) (at 171.45 104.14 90) (fields_autoplaced)
@@
       (effects (font (size 1.27 1.27)) (justify left))
     )
-    (pin "GND" output (at 208.28 106.68 180)
-      (effects (font (size 1.27 1.27)) (justify left))
-    )
+    (pin "GND" output (at 208.28 105.41 180)
+      (effects (font (size 1.27 1.27)) (justify left))
+    )

Commit message: Add files via upload
Parts:
- added J24, J26: Conn_02x04_Odd_Even, Connector_IDC:IDC-Header_2x04_P2.54mm_Vertical, symbol Connector_Generic:Conn_02x04_Odd_Even
- J10: footprint (none) -> Connector_JST:JST_EH_S3B-EH_1x03_P2.50mm_Horizontal
- JP2: footprint (none) -> Jumper:SolderJumper-2_P1.3mm_Open_RoundedPad1.0x1.5mm
- R29: footprint (none) -> Resistor_SMD:R_0603_1608Metric_Pad0.98x0.95mm_HandSolder
Connections:
- new net Current_Sense1: J24.2 (Pin_2)
- new net Current_Sense2: J24.4 (Pin_4)
- new net Current_Sense3: J26.2 (Pin_2)
- new net Current_Sense4: J26.4 (Pin_4)
- new net INA_M1_BACK: J26.1 (Pin_1)
- new net INA_M1_FRONT: J24.1 (Pin_1)
- new net INA_M2_BACK: J26.7 (Pin_7)
- new net INA_M2_FRONT: J24.7 (Pin_7)
- new net INB_M1_BACK: J26.3 (Pin_3)
- new net INB_M1_FRONT: J24.3 (Pin_3)
- new net INB_M2_BACK: J26.6 (Pin_6)
- new net INB_M2_FRONT: J24.6 (Pin_6)
- new net PWM_M1_BACK: J26.5 (Pin_5)
- new net PWM_M1_FRONT: J24.5 (Pin_5)
- new net PWM_M2_BACK: J26.8 (Pin_8)
- new net PWM_M2_FRONT: J24.8 (Pin_8)
Other:
- added sheet ENCODER (ENCODER.kicad_sch)
- sheet Esp_1 ports: added HALL_IN; removed none
- sheet Esp_2 ports: added A_LEFT, A_RIGHT, B_LEFT, B_RIGHT, Current_Sense_1, Current_Sense_2, Current_Sense_3, Current_Sense_4, INA_M1_BACK, INA_M1_FRONT, INA_M2_BACK, INA_M2_FRONT, INB_M1_BACK, INB_M1_FRONT, INB_M2_BACK, INB_M2_FRONT, PWM_M1_BACK, PWM_M1_FRONT, PWM_M2_BACK, PWM_M2_FRONT, RX_2, TX_2; removed none
- sheet SENSORES ports: added 5V, HALL_OUT, SCL, SDA; removed 3,3V

Commit message: Add files via upload
Parts:
- removed J24, J26: Conn_02x04_Odd_Even, Connector_IDC:IDC-Header_2x04_P2.54mm_Vertical, symbol Connector_Generic:Conn_02x04_Odd_Even
- added J2, J3: Conn_02x07_Counter_Clockwise, Connector_IDC:IDC-Header_2x07_P2.54mm_Vertical, symbol Connector_Generic:Conn_02x07_Counter_Clockwise
Connections:
- net LED_LVL_SHIFTER/EXT_5V is gone; now on net Esp1_5V: J10.2 (Pin_2)
- net Current_Sense1: now also J3.14 (Pin_14)
- net Current_Sense2: now also J3.12 (Pin_12)
- net Current_Sense3: now also J2.14 (Pin_14)
- net Current_Sense4: now also J2.12 (Pin_12)
- net GND: now also J2.11 (Pin_11), J2.13 (Pin_13), J2.2 (Pin_2), J2.4 (Pin_4), J2.6 (Pin_6), J2.9 (Pin_9), J3.11 (Pin_11), J3.13 (Pin_13), J3.2 (Pin_2), J3.4 (Pin_4), J3.6 (Pin_6), J3.9 (Pin_9)
- net INA_M1_BACK: now also J2.1 (Pin_1)
- net INA_M1_FRONT: now also J3.1 (Pin_1)
- net INA_M2_BACK: now also J2.7 (Pin_7)
- net INA_M2_FRONT: now also J3.7 (Pin_7)
- net INB_M1_BACK: now also J2.3 (Pin_3)
- net INB_M1_FRONT: now also J3.3 (Pin_3)
- net INB_M2_BACK: now also J2.10 (Pin_10)
- net INB_M2_FRONT: now also J3.10 (Pin_10)
- net PWM_M1_BACK: now also J2.5 (Pin_5)
- net PWM_M1_FRONT: now also J3.5 (Pin_5)
- net PWM_M2_BACK: now also J2.8 (Pin_8)
- net PWM_M2_FRONT: now also J3.8 (Pin_8)
Other:
- sheet Esp_1 ports: added EXT_5V_1; removed EXT_5V
- sheet Esp_2 ports: added 3,3V_ESP2, EXT_5V_2; removed EXT_5V

Commit message: Add files via upload
Parts:
- removed J2, J3: Conn_02x07_Counter_Clockwise, Connector_IDC:IDC-Header_2x07_P2.54mm_Vertical, symbol Connector_Generic:Conn_02x07_Counter_Clockwise
- added J25: Conn_01x02, TerminalBlock_Phoenix:TerminalBlock_Phoenix_MKDS-3-2-5.08_1x02_P5.08mm_Horizontal, symbol Connector_Generic:Conn_01x02
Connections:
- net CANH: now also J25.2 (Pin_2)
- net CANL: now also J25.1 (Pin_1)
Other:
- removed sheet ENCODER
- removed sheet Esp_2
- removed sheet SN65HVD230_2
