File: fred_v3/Motors_Back.kicad_sch (KiCad schematic)
At the start: 24 parts, among them Q8 NMOS, Q9 NMOS, U16 VNH2SP30, U17 VNH2SP30

Commit message: Add files via upload
Parts:
- C43, C44, C45, C46, C47, C48: footprint Capacitor_SMD:C_0603_1608Metric_Pad1.08x0.95mm_HandSolder -> Capacitor_THT:C_Radial_D10.0mm_H20.0mm_P5.00mm
