File: fred_v3/POWER_POT.kicad_sch (KiCad schematic)
At the start: 34 parts, among them IC5 PAC1921-1-AIA-TR, J11 Conn_01x02, J32 Conn_01x06, J33 Conn_01x06, SW5 SW_DIP_x01, U11 L7805, U13 L7805

Commit message: Add files via upload
Parts:
- removed C30: 2,2uF, Capacitor_SMD:C_0603_1608Metric_Pad1.08x0.95mm_HandSolder, symbol Device:C
- removed C30 (x2): C, Capacitor_SMD:C_0603_1608Metric_Pad1.08x0.95mm_HandSolder, symbol Device:C
- removed C31: 0,1uF, Capacitor_SMD:C_0603_1608Metric_Pad1.08x0.95mm_HandSolder, symbol Device:C
- removed D23: BPC_M1, LED_SMD:LED_1206_3216Metric_Pad1.42x1.75mm_HandSolder, symbol Device:LED
- removed D24: E2C, LED_SMD:LED_1206_3216Metric_Pad1.42x1.75mm_HandSolder, symbol Device:LED
- removed D24: E1C, LED_SMD:LED_1206_3216Metric_Pad1.42x1.75mm_HandSolder, symbol Device:LED
- removed F1 (x2): Fuse 40Amp, Fuse:Fuseholder_Clip-5x20mm_Littelfuse_111_Inline_P20.00x5.00mm_D1.05mm_Horizontal, symbol Device:Fuse
- removed F5: Fuse 1Amp, Fuse:Fuseholder_Clip-6.3x32mm_Littelfuse_102_Inline_P34.21x7.62mm_D2.54mm_Horizontal, symbol Device:Fuse
- removed IC5 (x2): PAC1921-1-AIA-TR, Package_DFN_QFN:WDFN-10-1EP_3x3mm_P0.5mm_EP1.8x2.5mm, symbol PAC1921:PAC1921-1-AIA-TR
- removed J11: Conn_01x02, Connector_AMASS:AMASS_XT60-M_1x02_P7.20mm_Vertical, symbol Connector_Generic:Conn_01x02
- removed J32, J33: Conn_01x06, Connector_JST:JST_EH_S6B-EH_1x06_P2.50mm_Horizontal, symbol Connector_Generic:Conn_01x06
- removed R108 (x2): R_Shunt, Resistor_SMD:R_0603_1608Metric_Pad0.98x0.95mm_HandSolder, symbol Device:R
- removed R109 (x2), R110 (x2): R, Resistor_SMD:R_0603_1608Metric_Pad0.98x0.95mm_HandSolder, symbol Device:R
- removed R111, R112 (x2): 330, Resistor_SMD:R_0603_1608Metric_Pad0.98x0.95mm_HandSolder, symbol Device:R
- removed SW5: SW_DIP_x01, Connector_AMASS:AMASS_XT60-M_1x02_P7.20mm_Vertical, symbol Switch:SW_DIP_x01
- removed U11: L7805, Package_TO_SOT_THT:TO-220-3_Horizontal_TabDown, symbol Regulator_Linear:L7805
- added C30: C, Capacitor_SMD:C_0603_1608Metric_Pad1.08x0.95mm_HandSolder, symbol Device:C
- added D24: E1C, LED_SMD:LED_1206_3216Metric_Pad1.42x1.75mm_HandSolder, symbol Device:LED
- added F1: Fuse 40Amp, Fuse:Fuseholder_Clip-5x20mm_Littelfuse_111_Inline_P20.00x5.00mm_D1.05mm_Horizontal, symbol Device:Fuse
- added IC5: PAC1921-1-AIA-TR, Package_DFN_QFN:WDFN-10-1EP_3x3mm_P0.5mm_EP1.8x2.5mm, symbol PAC1921:PAC1921-1-AIA-TR
- added R108: R_Shunt, Resistor_SMD:R_0603_1608Metric_Pad0.98x0.95mm_HandSolder, symbol Device:R
- added R109, R110: R, Resistor_SMD:R_0603_1608Metric_Pad0.98x0.95mm_HandSolder, symbol Device:R
- added R112: 330, Resistor_SMD:R_0603_1608Metric_Pad0.98x0.95mm_HandSolder, symbol Device:R
Connections:
- net 12V_IN: now also IC5.2 (SENSE+), R108.1
- net GND: now also C30.2, D24.1 (K), IC5.11 (EP), IC5.5 (GND), R110.2
- net Pot_5V_1: now also IC5.7 (RESERVED)
- net SENSED_12V: now also F1.1, R112.1
- new net: D24.2 (A), R112.2
- new net: C30.1, IC5.1 (VDD), R109.2
- new net: F1.2, IC5.3 (SENSE-), R108.2
- new net: IC5.6 (ADDR_SEL), R110.1
- new net Esp_3,3V: R109.1
- new net Esp_I2C_Clock: IC5.10 (SM_CLK)
- new net Esp_I2C_Data: IC5.9 (SM_DATA)
- new net Esp_R/W_PAC1921: IC5.8 (~{READ}/INT)
- no-connect marks 2 -> 1
Other:
- note removed: "LEDs indicadores"
- moved on the sheet: C60, C61, D23, F4, J11, R111, SW5, U13
