File: fred_v3/RASP.kicad_sch (KiCad schematic)
At the start: 18 parts, among them J12 Conn_02x20_Odd_Even, J13 FAN1, J14 FAN2, J15 FAN3, J16 FAN4, Q7 NMOS, U14 MCP2515-xSO, Y1 Crystal

Commit message: Add files via upload
Parts:
- added J29: Conn_02x20_Odd_Even, Connector_PinSocket_2.54mm:PinSocket_2x20_P2.54mm_Vertical, symbol Connector_Generic:Conn_02x20_Odd_Even
- added J34, J35: Conn_01x04, Connector_JST:JST_EH_S4B-EH_1x04_P2.50mm_Horizontal, symbol Connector_Generic:Conn_01x04
- C37, C38, C39, C40: footprint (none) -> Capacitor_SMD:C_0603_1608Metric_Pad1.08x0.95mm_HandSolder
- D15: footprint (none) -> Diode_SMD:D_SOD-128
- J12: footprint (none) -> Connector_PinSocket_2.54mm:PinSocket_2x20_P2.54mm_Vertical
- J13, J14, J15, J16: footprint (none) -> Connector_JST:JST_EH_B2B-EH-A_1x02_P2.50mm_Vertical
- Q7: footprint (none) -> Package_TO_SOT_SMD:TO-252-2
- R41, R42, R43, R44, R46: footprint (none) -> Resistor_SMD:R_0603_1608Metric_Pad0.98x0.95mm_HandSolder
- Y1: footprint (none) -> Crystal:Crystal_HC49-4H_Vertical
Connections:
- net 3,3V: now also J29.1 (Pin_1), J29.17 (Pin_17), J34.4 (Pin_4), J35.4 (Pin_4)
- net 5V: now also J29.2 (Pin_2), J29.4 (Pin_4)
- net GND: now also J29.14 (Pin_14), J29.20 (Pin_20), J29.25 (Pin_25), J29.30 (Pin_30), J29.34 (Pin_34), J29.39 (Pin_39), J29.6 (Pin_6), J29.9 (Pin_9), J34.3 (Pin_3), J35.3 (Pin_3)
- net GPIO0(ID_SD): now also J29.27 (Pin_27)
- net GPIO1(ID_SC): now also J29.28 (Pin_28)
- net GPIO10(MOSI): now also J29.19 (Pin_19)
- net GPIO11(SCLK): now also J29.23 (Pin_23)
- net GPIO12(PWM0): now also J29.32 (Pin_32)
- net GPIO13(PWM1): now also J29.33 (Pin_33)
- net GPIO14(TXD): now also J29.8 (Pin_8)
- net GPIO15(RXD): now also J29.10 (Pin_10)
- net GPIO16: now also J29.36 (Pin_36)
- net GPIO17: now also J29.11 (Pin_11)
- net GPIO18(PCM_CLK): now also J29.12 (Pin_12)
- net GPIO19(PCM_FS): now also J29.35 (Pin_35)
- net GPIO2(SDA): now also J29.3 (Pin_3), J34.2 (Pin_2), J35.2 (Pin_2)
- net GPIO20(PCM_DIN): now also J29.38 (Pin_38)
- net GPIO21(PCM_DOUT): now also J29.40 (Pin_40)
- net GPIO22: now also J29.15 (Pin_15)
- net GPIO23: now also J29.16 (Pin_16)
- net GPIO24: now also J29.18 (Pin_18)
- net GPIO25: now also J29.22 (Pin_22)
- net GPIO26: now also J29.37 (Pin_37)
- net GPIO27: now also J29.13 (Pin_13)
- net GPIO3(SCL): now also J29.5 (Pin_5), J34.1 (Pin_1), J35.1 (Pin_1)
- net GPIO4(GPCLK0): now also J29.7 (Pin_7)
- net GPIO5: now also J29.29 (Pin_29)
- net GPIO6: now also J29.31 (Pin_31)
- net GPIO7(CE1): now also J29.26 (Pin_26)
- net GPIO8(CE0): now also J29.24 (Pin_24)
- net GPIO9(MISO): now also J29.21 (Pin_21)
Other:
- moved on the sheet: C37, C38, C39, C40, D15, J12, J13, J14, J15, J16, Q7, R41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

Commit message: Add files via upload
Connections:
- net 5V: no longer J12.2 (Pin_2), J12.4 (Pin_4)
- new net Rasp_5V: J12.2 (Pin_2), J12.4 (Pin_4)
Changed lines of the file:
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@@
   (junction (at 30.48 97.79) (diameter 0) (color 0 0 0 0)
   )
+  (junction (at 264.16 57.15) (diameter 0) (color 0 0 0 0)
+  )
   (junction (at 238.76 53.34) (diameter 0) (color 0 0 0 0)
   )
@@
   )
   (junction (at 236.22 55.88) (diameter 0) (color 0 0 0 0)
-  )
-  (junction (at 265.43 57.15) (diameter 0) (color 0 0 0 0)
   )
   (junction (at 289.56 200.66) (diameter 0) (color 0 0 0 0)
@@
     (stroke (width 0) (type default))
   )
+  (wire (pts (xy 264.16 59.69) (xy 264.16 57.15))
+    (stroke (width 0) (type default))
+  )
   (wire (pts (xy 302.26 204.47) (xy 294.64 204.47))
     (stroke (width 0) (type default))
@@
     (stroke (width 0) (type default))
   )
+  (wire (pts (xy 261.62 59.69) (xy 264.16 59.69))
+    (stroke (width 0) (type default))
+  )
   (wire (pts (xy 100.33 58.42) (xy 100.33 60.96))
     (stroke (width 0) (type default))
@@
     (stroke (width 0) (type default))
   )
-  (wire (pts (xy 266.7 57.15) (xy 265.43 57.15))
+  (wire (pts (xy 264.16 57.15) (xy 261.62 57.15))
     (stroke (width 0) (type default))
   )
@@
     (stroke (width 0) (type default))
   )
-  (wire (pts (xy 265.43 57.15) (xy 261.62 57.15))
+  (wire (pts (xy 265.43 57.15) (xy 264.16 57.15))
     (stroke (width 0) (type default))
   )
@@
     )
   )
-  (global_label "5V" (shape input) (at 266.7 57.15 0) (fields_autoplaced)
-    (effects (font (size 1.27 1.27)) (justify left))
-    (property "Intersheetrefs" "${INTERSHEET_REFS}" (at 271.9833 57.15 0)
-      (effects (font (size 1.27 1.27)) (justify left) hide)
-    )
-  )
   (global_label "GPIO15(RXD)" (shape input) (at 344.17 68.58 0) (fields_autoplaced)
     (effects (font (size 1.27 1.27)) (justify left))
@@
     )
   )
-  (global_label "5V" (shape input) (at 261.62 59.69 0) (fields_autoplaced)
-    (effects (font (size 1.27 1.27)) (justify left))
-    (property "Intersheetrefs" "${INTERSHEET_REFS}" (at 266.9033 59.69 0)
-      (effects (font (size 1.27 1.27)) (justify left) hide)
-    )
-  )

Commit message: Add files via upload
Parts:
- removed J34, J35: Conn_01x04, Connector_JST:JST_EH_S4B-EH_1x04_P2.50mm_Horizontal, symbol Connector_Generic:Conn_01x04
Changed lines of the file:
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@@
-    (effects (font (size 1.27 1.27)) (justify right))
-  )
-  (hierarchical_label "Rasp_SDA" (shape input) (at 279.4 30.48 270) (fields_autoplaced)
     (effects (font (size 1.27 1.27)) (justify right))
   )
@@
     (effects (font (size 1.27 1.27)) (justify left))
   )
-  (hierarchical_label "Rasp_SCL" (shape input) (at 262.89 30.48 270) (fields_autoplaced)
-    (effects (font (size 1.27 1.27)) (justify right))
-  )
   (hierarchical_label "12V" (shape input) (at 267.97 167.64 90) (fields_autoplaced)
     (effects (font (size 1.27 1.27)) (justify left))
@@
     (effects (font (size 1.27 1.27)) (justify left))
   )
-  (hierarchical_label "Rasp_3,3V" (shape input) (at 270.51 30.48 270) (fields_autoplaced)
-    (effects (font (size 1.27 1.27)) (justify right))
-  )
-  (hierarchical_label "Rasp_3,3V" (shape input) (at 284.48 30.48 270) (fields_autoplaced)
-    (effects (font (size 1.27 1.27)) (justify right))
-  )
-  (hierarchical_label "Rasp_SDA" (shape input) (at 265.43 30.48 270) (fields_autoplaced)
-    (effects (font (size 1.27 1.27)) (justify right))
-  )
-  (hierarchical_label "Rasp_SCL" (shape input) (at 276.86 30.48 270) (fields_autoplaced)
-    (effects (font (size 1.27 1.27)) (justify right))
-  )
   (hierarchical_label "Rasp_5V" (shape input) (at 267.97 54.61 0) (fields_autoplaced)
     (effects (font (size 1.27 1.27)) (justify left))
@@
         (path "/210292b2-d6ba-424c-bd40-e4a2be18eb8d/5bbeae27-92ef-458a-a66f-e2aa3c6ef98a"
           (reference "R46") (unit 1)
-        )
-      )
-    )
-  )
-  (symbol (lib_id "Connector_Generic:Conn_01x04") (at 265.43 25.4 90) (unit 1)
-    (in_bom yes) (on_board yes) (dnp no) (fields_autoplaced)
-    (property "Reference" "J34" (at 266.7 19.05 90)
-      (effects (font (size 1.27 1.27)))
-    )
-    (property "Value" "Conn_01x04" (at 266.7 21.59 90)
-      (effects (font (size 1.27 1.27)))
-    )
-    (property "Footprint" "Connector_JST:JST_EH_S4B-EH_1x04_P2.50mm_Horizontal" (at 265.43 25.4 0)
-      (effects (font (size 1.27 1.27)) hide)
-    )
-    (property "Datasheet" "~" (at 265.43 25.4 0)
-      (effects (font (size 1.27 1.27)) hide)
-    )
-    (pin "1")
-    (pin "2")
-    (pin "3")
-    (pin "4")
-    (instances
-      (project "fred_v3"
-        (path "/210292b2-d6ba-424c-bd40-e4a2be18eb8d/5bbeae27-92ef-458a-a66f-e2aa3c6ef98a"
-          (reference "J34") (unit 1)
         )
       )
@@
     )
   )
-  (symbol (lib_id "power:GND") (at 281.94 30.48 0) (unit 1)
-    (in_bom yes) (on_board yes) (dnp no) (fields_autoplaced)
-    (property "Reference" "#PWR0158" (at 281.94 36.83 0)
-      (effects (font (size 1.27 1.27)) hide)
-    )
-    (property "Value" "GND" (at 281.94 35.56 0)
-      (effects (font (size 1.27 1.27)))
-    )
-    (property "Footprint" "" (at 281.94 30.48 0)
-      (effects (font (size 1.27 1.27)) hide)
-    )
-    (property "Datasheet" "" (at 281.94 30.48 0)
-      (effects (font (size 1.27 1.27)) hide)
-    )
-    (pin "1")
-    (instances
-      (project "fred_v3"
-        (path "/210292b2-d6ba-424c-bd40-e4a2be18eb8d/5bbeae27-92ef-458a-a66f-e2aa3c6ef98a"
-          (reference "#PWR0158") (unit 1)
-        )
-      )
-    )
-  )
   (symbol (lib_id "Device:R") (at 128.27 88.9 0) (unit 1)
     (in_bom yes) (on_board yes) (dnp no) (fields_autoplaced)
@@
         )
       )
-    )
-  )
-  (symbol (lib_id "power:GND") (at 267.97 30.48 0) (unit 1)
-    (in_bom yes) (on_board yes) (dnp no) (fields_autoplaced)
-    (property "Reference" "#PWR0157" (at 267.97 36.83 0)
-      (effects (font (size 1.27 1.27)) hide)
-    )
-    (property "Value" "GND" (at 267.97 35.56 0)
-      (effects (font (size 1.27 1.27)))
-    )
-    (property "Footprint" "" (at 267.97 30.48 0)
-      (effects (font (size 1.27 1.27)) hide)
-    )
-    (property "Datasheet" "" (at 267.97 30.48 0)
-      (effects (font (size 1.27 1.27)) hide)
-    )
-    (pin "1")
-    (instances
-      (project "fred_v3"
-        (path "/210292b2-d6ba-424c-bd40-e4a2be18eb8d/5bbeae27-92ef-458a-a66f-e2aa3c6ef98a"
-          (reference "#PWR0157") (unit 1)
-        )
-      )
-    )
-  )
-  (symbol (lib_id "Connector_Generic:Conn_01x04") (at 279.4 25.4 90) (unit 1)
-    (in_bom yes) (on_board yes) (dnp no) (fields_autoplaced)
-    (property "Reference" "J35" (at 280.67 19.05 90)
-      (effects (font (size 1.27 1.27)))
-    )
-    (property "Value" "Conn_01x04" (at 280.67 21.59 90)
-      (effects (font (size 1.27 1.27)))
-    )
-    (property "Footprint" "Connector_JST:JST_EH_S4B-EH_1x04_P2.50mm_Horizontal" (at 279.4 25.4 0)
-      (effects (font (size 1.27 1.27)) hide)
-    )
-    (property "Datasheet" "~" (at 279.4 25.4 0)
-      (effects (font (size 1.27 1.27)) hide)
-    )
-    (pin "1")
-    (pin "2")
-    (pin "3")
-    (pin "4")
-    (instances
-      (project "fred_v3"
-        (path "/210292b2-d6ba-424c-bd40-e4a2be18eb8d/5bbeae27-92ef-458a-a66f-e2aa3c6ef98a"
-          (reference "J35") (unit 1)
-        )
-      )
