File: fred_v3/fred_v3.kicad_sch (KiCad schematic)
At the start: 0 parts

Commit message: Add files via upload
Other:
- added sheet RASP (RASP.kicad_sch)
- sheet Lógica ports: added CANH, CANL, Esp1_5V, Esp2_5V, GND; removed none
- sheet POWER ports: added Esp1_5V, Esp2_5V, GND, Rasp_3,3V, Rasp_5V, Rasp_I2C_Clock, Rasp_I2C_Data, Rasp_R/W_PAC1921, S_12V; removed none
- note added: "Bateria, proteção, monitoramento de tensão/corrente/potência via I2C e regulagem de tensão."
Changed lines of the file:
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@@
     (company "FRED")
   )
-  (sheet (at 110.49 68.58) (size 58.42 49.53) (fields_autoplaced)
+  (junction (at 107.95 104.14) (diameter 0) (color 0 0 0 0)
+  )
+  (wire (pts (xy 107.95 104.14) (xy 119.38 104.14))
+    (stroke (width 0) (type default))
+  )
+  (wire (pts (xy 119.38 40.64) (xy 107.95 40.64))
+    (stroke (width 0) (type default))
+  )
+  (wire (pts (xy 96.52 101.6) (xy 119.38 101.6))
+    (stroke (width 0) (type default))
+  )
+  (wire (pts (xy 59.69 35.56) (xy 119.38 35.56))
+    (stroke (width 0) (type default))
+  )
+  (wire (pts (xy 57.15 91.44) (xy 57.15 33.02))
+    (stroke (width 0) (type default))
+  )
+  (wire (pts (xy 119.38 30.48) (xy 54.61 30.48))
+    (stroke (width 0) (type default))
+  )
+  (wire (pts (xy 96.52 104.14) (xy 107.95 104.14))
+    (stroke (width 0) (type default))
+  )
+  (wire (pts (xy 59.69 91.44) (xy 59.69 35.56))
+    (stroke (width 0) (type default))
+  )
+  (wire (pts (xy 143.51 76.2) (xy 143.51 91.44))
+    (stroke (width 0) (type default))
+  )
+  (wire (pts (xy 140.97 76.2) (xy 140.97 91.44))
+    (stroke (width 0) (type default))
+  )
+  (wire (pts (xy 107.95 40.64) (xy 107.95 104.14))
+    (stroke (width 0) (type default))
+  )
+  (wire (pts (xy 62.23 91.44) (xy 62.23 38.1))
+    (stroke (width 0) (type default))
+  )
+  (wire (pts (xy 62.23 38.1) (xy 119.38 38.1))
+    (stroke (width 0) (type default))
+  )
+  (wire (pts (xy 96.52 99.06) (xy 119.38 99.06))
+    (stroke (width 0) (type default))
+  )
+  (wire (pts (xy 57.15 33.02) (xy 119.38 33.02))
+    (stroke (width 0) (type default))
+  )
+  (wire (pts (xy 54.61 30.48) (xy 54.61 91.44))
+    (stroke (width 0) (type default))
+  )
+  (text "Bateria, proteção, monitoramento de \ntensão/corrente/potência via I2C e regulagem de tensão."
+    (at 38.1 87.63 0)
+    (effects (font (size 1.27 1.27)) (justify left bottom))
+  )
+  (sheet (at 119.38 91.44) (size 58.42 49.53) (fields_autoplaced)
     (stroke (width 0.1524) (type solid))
     (fill (color 0 0 0 0.0000))
-    (property "Sheetname" "Lógica" (at 110.49 67.8684 0)
+    (property "Sheetname" "Lógica" (at 119.38 90.7284 0)
       (effects (font (size 1.27 1.27)) (justify left bottom))
     )
-    (property "Sheetfile" "Lógica.kicad_sch" (at 110.49 118.6946 0)
+    (property "Sheetfile" "Lógica.kicad_sch" (at 119.38 141.5546 0)
       (effects (font (size 1.27 1.27)) (justify left top))
+    )
+    (pin "Esp1_5V" input (at 119.38 99.06 180)
+      (effects (font (size 1.27 1.27)) (justify left))
+    )
+    (pin "CANL" input (at 143.51 91.44 90)
+      (effects (font (size 1.27 1.27)) (justify right))
+    )
+    (pin "CANH" input (at 140.97 91.44 90)
+      (effects (font (size 1.27 1.27)) (justify right))
+    )
+    (pin "Esp2_5V" input (at 119.38 101.6 180)
+      (effects (font (size 1.27 1.27)) (justify left))
+    )
+    (pin "GND" input (at 119.38 104.14 180)
+      (effects (font (size 1.27 1.27)) (justify left))
     )
     (instances
@@
     )
   )
-  (sheet (at 29.21 68.58) (size 58.42 49.53) (fields_autoplaced)
+  (sheet (at 119.38 26.67) (size 59.69 49.53)
     (stroke (width 0.1524) (type solid))
     (fill (color 0 0 0 0.0000))
-    (property "Sheetname" "POWER" (at 29.21 67.8684 0)
+    (property "Sheetname" "RASP" (at 119.38 25.9584 0)
       (effects (font (size 1.27 1.27)) (justify left bottom))
     )
-    (property "Sheetfile" "POWER.kicad_sch" (at 29.21 118.6946 0)
+    (property "Sheetfile" "RASP.kicad_sch" (at 115.57 77.47 0)
       (effects (font (size 1.27 1.27)) (justify left top))
+    )
+    (pin "Rasp_5V" input (at 119.38 33.02 180)
+      (effects (font (size 1.27 1.27)) (justify left))
+    )
+    (pin "Rasp_SCL" input (at 119.38 35.56 180)
+      (effects (font (size 1.27 1.27)) (justify left))
+    )
+    (pin "Rasp_SDA" input (at 119.38 38.1 180)
+      (effects (font (size 1.27 1.27)) (justify left))
+    )
+    (pin "GND" input (at 119.38 40.64 180)
+      (effects (font (size 1.27 1.27)) (justify left))
+    )
+    (pin "Rasp_3,3V" input (at 119.38 30.48 180)
+      (effects (font (size 1.27 1.27)) (justify left))
+    )
+    (pin "CANH" input (at 140.97 76.2 270)
+      (effects (font (size 1.27 1.27)) (justify left))
+    )
+    (pin "CANL" input (at 143.51 76.2 270)
+      (effects (font (size 1.27 1.27)) (justify left))
+    )
+    (instances
+      (project "fred_v3"
+        (path "/210292b2-d6ba-424c-bd40-e4a2be18eb8d" (page "12"))
+      )
+    )
+  )
+  (sheet (at 38.1 91.44) (size 58.42 49.53) (fields_autoplaced)
+    (stroke (width 0.1524) (type solid))
+    (fill (color 0 0 0 0.0000))
+    (property "Sheetname" "POWER" (at 38.1 90.7284 0)
+      (effects (font (size 1.27 1.27)) (justify left bottom))
+    )
+    (property "Sheetfile" "POWER.kicad_sch" (at 38.1 141.5546 0)
+      (effects (font (size 1.27 1.27)) (justify left top))
+    )
+    (pin "Rasp_I2C_Data" input (at 62.23 91.44 90)
+      (effects (font (size 1.27 1.27)) (justify right))
+    )
+    (pin "Rasp_I2C_Clock" input (at 59.69 91.44 90)
+      (effects (font (size 1.27 1.27)) (justify right))
+    )
+    (pin "Rasp_R{slash}W_PAC1921" input (at 64.77 91.44 90)
+      (effects (font (size 1.27 1.27)) (justify right))
+    )
+    (pin "Esp1_5V" input (at 96.52 99.06 0)
+      (effects (font (size 1.27 1.27)) (justify right))
+    )
+    (pin "Rasp_5V" input (at 57.15 91.44 90)
+      (effects (font (size 1.27 1.27)) (justify right))
+    )
+    (pin "Esp2_5V" input (at 96.52 101.6 0)
+      (effects (font (size 1.27 1.27)) (justify right))
+    )
+    (pin "GND" input (at 96.52 104.14 0)
+      (effects (font (size 1.27 1.27)) (justify right))
+    )
+    (pin "Rasp_3,3V" input (at 54.61 91.44 90)
+      (effects (font (size 1.27 1.27)) (justify right))
+    )
+    (pin "S_12V" input (at 67.31 91.44 90)
+      (effects (font (size 1.27 1.27)) (justify right))
     )
     (instances
@@
     )
   )
-  (sheet (at 189.23 68.58) (size 59.69 49.53) (fields_autoplaced)
+  (sheet (at 198.12 91.44) (size 59.69 49.53) (fields_autoplaced)
     (stroke (width 0.1524) (type solid))
     (fill (color 0 0 0 0.0000))
-    (property "Sheetname" "Potência" (at 189.23 67.8684 0)
+    (property "Sheetname" "Potência" (at 198.12 90.7284 0)
       (effects (font (size 1.27 1.27)) (justify left bottom))
     )
-    (property "Sheetfile" "Potência.kicad_sch" (at 189.23 118.6946 0)
+    (property "Sheetfile" "Potência.kicad_sch" (at 198.12 141.5546 0)
       (effects (font (size 1.27 1.27)) (justify left top))
     )

Commit message: Add files via upload
Other:
- added sheet POWER_POT (POWER_POT.kicad_sch)
- sheet Potência ports: added 12V, 5V_1, 5V_2, GND; removed none
- sheet RASP ports: added 12V, Rasp_R/W_PAC1921_LOG; removed none
Changed lines of the file:
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@@
   (paper "A4")
   (title_block
+    (rev "1")
     (company "FRED")
   )
@@
     (stroke (width 0) (type default))
   )
+  (wire (pts (xy 67.31 91.44) (xy 67.31 43.18))
+    (stroke (width 0) (type default))
+  )
   (wire (pts (xy 96.52 101.6) (xy 119.38 101.6))
     (stroke (width 0) (type default))
   )
+  (wire (pts (xy 67.31 43.18) (xy 119.38 43.18))
+    (stroke (width 0) (type default))
+  )
   (wire (pts (xy 59.69 35.56) (xy 119.38 35.56))
     (stroke (width 0) (type default))
   )
+  (wire (pts (xy 64.77 45.72) (xy 64.77 91.44))
+    (stroke (width 0) (type default))
+  )
   (wire (pts (xy 57.15 91.44) (xy 57.15 33.02))
     (stroke (width 0) (type default))
   )
-  (wire (pts (xy 119.38 30.48) (xy 54.61 30.48))
+  (wire (pts (xy 54.61 30.48) (xy 119.38 30.48))
+    (stroke (width 0) (type default))
+  )
+  (wire (pts (xy 243.84 76.2) (xy 243.84 91.44))
+    (stroke (width 0) (type default))
+  )
+  (wire (pts (xy 119.38 45.72) (xy 64.77 45.72))
     (stroke (width 0) (type default))
   )
@@
     (stroke (width 0) (type default))
   )
+  (wire (pts (xy 241.3 76.2) (xy 241.3 91.44))
+    (stroke (width 0) (type default))
+  )
   (wire (pts (xy 96.52 99.06) (xy 119.38 99.06))
     (stroke (width 0) (type default))
@@
     (stroke (width 0) (type default))
   )
+  (wire (pts (xy 246.38 76.2) (xy 246.38 91.44))
+    (stroke (width 0) (type default))
+  )
   (wire (pts (xy 54.61 30.48) (xy 54.61 91.44))
+    (stroke (width 0) (type default))
+  )
+  (wire (pts (xy 238.76 76.2) (xy 238.76 91.44))
     (stroke (width 0) (type default))
   )
@@
       (effects (font (size 1.27 1.27)) (justify left))
     )
+    (pin "12V" input (at 119.38 43.18 180)
+      (effects (font (size 1.27 1.27)) (justify left))
+    )
+    (pin "Rasp_R{slash}W_PAC1921_LOG" input (at 119.38 45.72 180)
+      (effects (font (size 1.27 1.27)) (justify left))
+    )
     (instances
       (project "fred_v3"
@@
     )
   )
+  (sheet (at 198.12 26.67) (size 58.42 49.53) (fields_autoplaced)
+    (stroke (width 0.1524) (type solid))
+    (fill (color 0 0 0 0.0000))
+    (property "Sheetname" "POWER_POT" (at 198.12 25.9584 0)
+      (effects (font (size 1.27 1.27)) (justify left bottom))
+    )
+    (property "Sheetfile" "POWER_POT.kicad_sch" (at 198.12 76.7846 0)
+      (effects (font (size 1.27 1.27)) (justify left top))
+    )
+    (pin "GND" input (at 238.76 76.2 270)
+      (effects (font (size 1.27 1.27)) (justify left))
+    )
+    (pin "S_12V" input (at 241.3 76.2 270)
+      (effects (font (size 1.27 1.27)) (justify left))
+    )
+    (pin "Pot_5V_1" input (at 243.84 76.2 270)
+      (effects (font (size 1.27 1.27)) (justify left))
+    )
+    (pin "Pot_5V_2" input (at 246.38 76.2 270)
+      (effects (font (size 1.27 1.27)) (justify left))
+    )
+    (instances
+      (project "fred_v3"
+        (path "/210292b2-d6ba-424c-bd40-e4a2be18eb8d" (page "17"))
+        (path "/210292b2-d6ba-424c-bd40-e4a2be18eb8d/b54a5b77-6097-4562-9836-27b2c01ae506" (page "17"))
+      )
+    )
+  )
   (sheet (at 198.12 91.44) (size 59.69 49.53) (fields_autoplaced)
     (stroke (width 0.1524) (type solid))
@@
       (effects (font (size 1.27 1.27)) (justify left top))
     )
-    (instances
+    (pin "5V_2" input (at 246.38 91.44 90)
+      (effects (font (size 1.27 1.27)) (justify right))
+    )
+    (pin "12V" input (at 241.3 91.44 90)
+      (effects (font (size 1.27 1.27)) (justify right))
+    )
+    (pin "5V_1" input (at 243.84 91.44 90)
+      (effects (font (size 1.27 1.27)) (justify right))
+    )
+    (pin "GND" input (at 238.76 91.44 90)
+      (effects (font (size 1.27 1.27)) (justify right))
+    )
+    (instances

Commit message: Add files via upload
Other:
- sheet POWER_POT ports: added Esp_3,3V, Esp_I2C_Clock, Esp_I2C_Data, Esp_R/W_PAC1921; removed Pot_5V_1
- sheet Potência ports: added 3,3V_ESP3, ESP_3_SCL, ESP_3_SDA, Esp_R/W_PAC1921; removed 5V_1
Changed lines of the file:
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@@
+    (stroke (width 0) (type default))
+  )
+  (wire (pts (xy 228.6 76.2) (xy 228.6 91.44))
     (stroke (width 0) (type default))
   )
@@
     (stroke (width 0) (type default))
   )
-  (wire (pts (xy 243.84 76.2) (xy 243.84 91.44))
-    (stroke (width 0) (type default))
-  )
   (wire (pts (xy 119.38 45.72) (xy 64.77 45.72))
     (stroke (width 0) (type default))
@@
     (stroke (width 0) (type default))
   )
+  (wire (pts (xy 234.95 76.2) (xy 234.95 91.44))
+    (stroke (width 0) (type default))
+  )
   (wire (pts (xy 143.51 76.2) (xy 143.51 91.44))
     (stroke (width 0) (type default))
@@
     (stroke (width 0) (type default))
   )
+  (wire (pts (xy 231.14 76.2) (xy 231.14 91.44))
+    (stroke (width 0) (type default))
+  )
   (wire (pts (xy 96.52 99.06) (xy 119.38 99.06))
     (stroke (width 0) (type default))
   )
   (wire (pts (xy 57.15 33.02) (xy 119.38 33.02))
+    (stroke (width 0) (type default))
+  )
+  (wire (pts (xy 226.06 76.2) (xy 226.06 91.44))
     (stroke (width 0) (type default))
   )
@@
       (effects (font (size 1.27 1.27)) (justify left))
     )
-    (pin "Pot_5V_1" input (at 243.84 76.2 270)
-      (effects (font (size 1.27 1.27)) (justify left))
-    )
     (pin "Pot_5V_2" input (at 246.38 76.2 270)
+      (effects (font (size 1.27 1.27)) (justify left))
+    )
+    (pin "Esp_3,3V" input (at 234.95 76.2 270)
+      (effects (font (size 1.27 1.27)) (justify left))
+    )
+    (pin "Esp_R{slash}W_PAC1921" input (at 231.14 76.2 270)
+      (effects (font (size 1.27 1.27)) (justify left))
+    )
+    (pin "Esp_I2C_Data" input (at 228.6 76.2 270)
+      (effects (font (size 1.27 1.27)) (justify left))
+    )
+    (pin "Esp_I2C_Clock" input (at 226.06 76.2 270)
       (effects (font (size 1.27 1.27)) (justify left))
     )
@@
       (effects (font (size 1.27 1.27)) (justify right))
     )
-    (pin "5V_1" input (at 243.84 91.44 90)
-      (effects (font (size 1.27 1.27)) (justify right))
-    )
     (pin "GND" input (at 238.76 91.44 90)
       (effects (font (size 1.27 1.27)) (justify right))
     )
+    (pin "ESP_3_SDA" input (at 228.6 91.44 90)
+      (effects (font (size 1.27 1.27)) (justify right))
+    )
+    (pin "ESP_3_SCL" input (at 226.06 91.44 90)
+      (effects (font (size 1.27 1.27)) (justify right))
+    )
+    (pin "3,3V_ESP3" input (at 234.95 91.44 90)
+      (effects (font (size 1.27 1.27)) (justify right))
+    )
+    (pin "Esp_R{slash}W_PAC1921" input (at 231.14 91.44 90)
+      (effects (font (size 1.27 1.27)) (justify right))
+    )
