File: Fred_PCB_testes/FPCB_Teste/Esp.kicad_sch (KiCad schematic)
At the start: 50 parts, among them J4 USB_C_Receptacle_USB2.0, J7 Conn_01x15, J8 Conn_01x15, Q1 Q_PMOS_GSD, Q2 SS8050-G, Q3 SS8050-G, SW1 SW_Push, SW2 SW_Push, U4 AMS1117-3.3, U5 CP2102N-Axx-xQFN28, U6 ESP32-WROOM-E

Commit message: Add files via upload
Parts:
- J8: footprint Connector_PinHeader_2.54mm:PinHeader_1x15_P2.54mm_Horizontal -> Connector_PinHeader_2.54mm:PinHeader_1x15_P2.54mm_Vertical
- U6: footprint PCM_Espressif:ESP32-WROOM-32E -> RF_Module:ESP32-WROOM-32
Changed lines of the file:
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@@
       (effects (font (size 1.27 1.27)) (justify left))
     )
-    (property "Footprint" "PCM_Espressif:ESP32-WROOM-32E" (at 292.1 156.21 0)
+    (property "Footprint" "RF_Module:ESP32-WROOM-32" (at 292.1 156.21 0)
       (effects (font (size 1.27 1.27)) hide)
     )
@@
       (effects (font (size 1.27 1.27)) (justify left) hide)
     )
-    (property "Footprint" "Connector_PinHeader_2.54mm:PinHeader_1x15_P2.54mm_Horizontal" (at 314.96 226.06 0)
-      (effects (font (size 1.27 1.27)) hide)
-    )
+    (property "Footprint" "Connector_PinHeader_2.54mm:PinHeader_1x15_P2.54mm_Vertical" (at 314.96 226.06 0)
+      (effects (font (size 1.27 1.27)) hide)
+    )
